File: MyClockProject/switchBox/switchBox.kicad_sch (KiCad schematic)
At the start: 20 parts, among them J1 RJ45, J2 USB_C_Receptacle_PowerOnly_6P, J6 Conn_01x16_Socket, J7 Conn_01x08_Socket, SW1 RotaryEncoder_Switch, SW2 S4_SW_Push, SW3 S3_SW_Push, SW4 S2_SW_Push, SW5 S1_SW_Push, SW6 MODE_SW_Push, U1 ESP32-WROOM-32, U3 SH-U12, U4 OLED_SSD1306_128x32_I2C

Commit message: コントロールボックスとモーター制御用の基盤設計を修正しました。（主にESP32ソケット幅変更）
Parts:
- SW1: footprint Rotary_Encoder:RotaryEncoder_Alps_EC12E-Switch_Vertical_H20mm -> RotaryEncoder Alps EC12D1524403:EC12D1524403
Changed lines of the file:
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@@
 			)
 		)
-		(property "Footprint" "Rotary_Encoder:RotaryEncoder_Alps_EC12E-Switch_Vertical_H20mm"
+		(property "Footprint" "RotaryEncoder Alps EC12D1524403:EC12D1524403"
 			(at 153.67 121.666 0)
 			(hide yes)
